File: MX8Mx_EVK_MIPI_CSI-TSC_HM5065-ADAPTER.kicad_pcb (KiCad board)
At the start: 2 copper layers, 40.4 x 40.5 mm, 15 parts, among them J1 1888863-4, J2 BM10NB_0.8_-24DS-0.4V_51_, U1 MIC5259-2.8YD5-TR

Commit message: Finish layout
Parts:
- removed the TP1 at (114.6, 100.6)
- removed the TP1 at (114.6, 93.8)
- added TP1: TestPoint, TestPoint:TestPoint_Pad_D1.0mm, F.Cu at (114.7, 100.6)
- J2: footprint BM10NB0824DS04V51 -> footprints:BM10NB0824DS04V51
- moved R2 51.8 mm to (137.6, 102.0)
- moved U1 47.6 mm to (120.5, 104.9)
- moved C2 47.5 mm to (124.2, 105.8)
- moved C3 42.9 mm to (124.2, 103.9)
- moved R1 42.6 mm to (117.6, 104.9), turned to 270 degrees
- moved C1 41.7 mm to (120.4, 102.1)
- moved TP2 3.18 mm to (114.7, 96.6)
- moved J2 1.00 mm to (138.4, 96.0)
Connections:
- net /CSI_DN2__SD_LVDS2_N renamed /CSI_D2_N
- net /CSI_DN3__SD_LVDS3_N renamed /CSI_D3_N
- net /CSI_DP2__SD_LVDS2_P renamed /CSI_D2_P
- net /CSI_DP3__SD_LVDS3_P renamed /CSI_D3_P
- J1 pad A2: /CSI_DN0__SD_LVDS0_N -> /CSI_D0_N
- J1 pad A3: /CSI_DP0__SD_LVDS0_P -> /CSI_D0_P
- J1 pad A5: /CSI_DN1__SD_LVDS1_N -> /CSI_D1_N
- J1 pad A6: /CSI_DP1__SD_LVDS1_P -> /CSI_D1_P
- J1 pad B2: /CSI_CLK_N__SPCLK_LVDS0_N -> /CSI_CLK_N
- J1 pad B3: /CSI_CLK_P__SPCLK_LVDS0_P -> /CSI_CLK_P
- J2 pad 10: /CSI_nRST_1V8 -> /CSI_D0_P
- J2 pad 11: GND -> Net-(J2-Pad11)
- J2 pad 12: /CSI_MCLK_1V8 -> GND
- J2 pad 14: /CSI_DP1__SD_LVDS1_P -> /CSI_CLK_N
- J2 pad 15: /CSI_DN1__SD_LVDS1_N -> /I2C_SCL_1V8
- J2 pad 16: GND -> /CSI_CLK_P
- J2 pad 17: /CSI_CLK_P__SPCLK_LVDS0_P -> /I2C_SDA_1V8
- J2 pad 18: /CSI_CLK_N__SPCLK_LVDS0_N -> GND
- J2 pad 19: GND -> /CSI_nRST_1V8
- J2 pad 2: +2V8 -> +1V8
- J2 pad 20: /CSI_DP0__SD_LVDS0_P -> /CSI_D1_N
- J2 pad 21: /CSI_DN0__SD_LVDS0_N -> GND
- J2 pad 22: GND -> /CSI_D1_P
- J2 pad 23: /CSI_PWDN_1V8 -> /CSI_MCLK_1V8
- J2 pad 24: +1V8 -> GND
- J2 pad 3: GND -> +2V8
- J2 pad 4: Net-(J2-Pad4) -> /CSI_PWDN_1V8
- J2 pad 5: Net-(J2-Pad5) -> GND
- J2 pad 6: Net-(J2-Pad6) -> GND
- J2 pad 7: GND -> /AF-2V8
- J2 pad 8: /I2C_SCL_1V8 -> /CSI_D0_N
- J2 pad 9: /I2C_SDA_1V8 -> Net-(J2-Pad9)
- R2 pad 1: +2V8 -> /AF-2V8
- R2 pad 2: Net-(J2-Pad4) -> +2V8
Routing:
- net GND: track 141.2 -> 222.5 mm, vias 10 -> 47
- net /CSI_D0_N: track 0.00 -> 40.9 mm, vias 0 -> 2
- net /CSI_D0_P: track 0.00 -> 38.1 mm, vias 0 -> 2
- net /CSI_D1_N: track 0.00 -> 31.9 mm, vias 0 -> 2
- net /CSI_D1_P: track 0.00 -> 31.2 mm, vias 0 -> 2
- net /CSI_CLK_N: track 0.00 -> 30.6 mm
- net +2V8: track 0.00 -> 30.5 mm
- net +1V8: track 0.00 -> 28.0 mm
- net /CSI_D3_P: track 28.8 -> 1.80 mm
- net /CSI_CLK_P: track 0.00 -> 26.8 mm
- net /CSI_DN0__SD_LVDS0_N: track 26.2 -> 0.00 mm, vias 1 -> 0
- net /CSI_DP0__SD_LVDS0_P: track 26.1 -> 0.00 mm, vias 1 -> 0
- net /CSI_D2_N: track 27.7 -> 1.83 mm
- net /CSI_D3_N: track 28.5 -> 2.82 mm
- net /CSI_DN1__SD_LVDS1_N: track 25.1 -> 0.00 mm, vias 1 -> 0
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- added copper zone on B.Cu, net GND
- added copper zone on F.Cu, net GND
