File: MX8Mx_EVK_MIPI_CSI-TSC_HM5065-ADAPTER.sch (KiCad schematic (older format))
At the start: 17 parts, among them J1 1888863-4, J2 BM10NB_0.8_-24DS-0.4V_51_, U1 MIC5259-2.8YD5-TR

Commit message: Finish layout
Parts:
- removed TP3, TP4, TP5: TestPoint, TestPoint:TestPoint_Pad_D1.0mm, symbol Connector:TestPoint
Connections:
- net labels added: AF-2V8, CSI_CLK_N, CSI_CLK_P, CSI_D0_N, CSI_D0_P, CSI_D1_N, CSI_D1_P, CSI_D2_N, CSI_D2_P, CSI_D3_N, CSI_D3_P
- net labels removed: CSI_CLK_N__SPCLK_LVDS0_N, CSI_CLK_P__SPCLK_LVDS0_P, CSI_DN0__SD_LVDS0_N, CSI_DN1__SD_LVDS1_N, CSI_DN2__SD_LVDS2_N, CSI_DN3__SD_LVDS3_N, CSI_DP0__SD_LVDS0_P, CSI_DP1__SD_LVDS1_P, CSI_DP2__SD_LVDS2_P, CSI_DP3__SD_LVDS3_P
- wire segments 120 -> 116
Other:
- note added: "1"
- note added: "10"
- note added: "11"
- note added: "12"
- note added: "13"
- note added: "14"
- note added: "15"
- note added: "16"
- note added: "17"
- note added: "18"
- note added: "19"
- note added: "2"
- note added: "20"
- note added: "21"
- note added: "22"
- note added: "23"
- note added: "24"
- note added: "3"
- note added: "4"
- note added: "5"
- note added: "6"
- note added: "7"
- note added: "8"
- note added: "9"
- moved on the sheet: C1, C2, C3, H1, H2, H3, H4, J2, R1, R2, U1
